File: pcb/GridBoard/Grid.sch (EAGLE design)
At the start: 0 parts

Commit message: Large progress on schematic, and created blank board file. Comparator circuit requires review and components must be labeled
Parts:
- added C1, C2, C3, C4: 10uF, 1_SparkFun-Capacitors:CAP_POL1206
- added D1, D10, D100, D101, D102, D103, D104, D105, D106, D107, D108, D109, D11, D110, D111, D112, D113, D114, D115, D116, D117, D118, D119, D12, D120, D121, D122, D123, D124, D125, D126, D127, D128, D129, D13, D130, D131, D132, D133, D134, D135, D136, D137, D138, D139, D14, D140, D141, D142, D143, D144, D145, D146, D147, D148, D149, D15, D150, D151, D152, D153, D154, D155, D156, D157, D158, D159, D16, D160, D161, D162, D163, D164, D165, D166, D167, D168, D169, D17, D170, D171, D172, D173, D174, D175, D176, D177, D178, D179, D18, D180, D181, D182, D183, D184, D185, D186, D187, D188, D189, D19, D190, D191, D192, D193, D194, D195, D196, D197, D198, D199, D2, D20, D200, D201, D202, D203, D204, D205, D206, D207, D208, D209, D21, D210, D211, D212, D213, D214, D215, D216, D217, D218, D219, D22, D220, D221, D222, D223, D224, D225, D226, D227, D228, D229, D23, D230, D231, D232, D233, D234, D235, D236, D237, D238, D239, D24, D240, D241, D242, D243, D244, D245, D246, D247, D248, D249, D25, D250, D251, D252, D253, D254, D255, D256, D26, D27, D28, D29, D3, D30, D31, D32, D33, D34, D35, D36, D37, D38, D39, D4, D40, D41, D42, D43, D44, D45, D46, D47, D48, D49, D5, D50, D51, D52, D53, D54, D55, D56, D57, D58, D59, D6, D60, D61, D62, D63, D64, D65, D66, D67, D68, D69, D7, D70, D71, D72, D73, D74, D75, D76, D77, D78, D79, D8, D80, D81, D82, D83, D84, D85, D86, D87, D88, D89, D9, D90, D91, D92, D93, D94, D95, D96, D97, D98, D99: (no value), 1_SparkFun-DiscreteSemi:DIODESOD
- added IC1: LMV358SOIC, 1_SparkFun-AnalogIC:LMV358SOIC
- added IC2: 74154DW, 74xx-us:74154DW
- added Q1, Q10, Q11, Q12, Q13, Q14, Q15, Q16, Q2, Q3, Q4, Q5, Q6, Q7, Q8, Q9: (no value), 1_SparkFun-DiscreteSemi:TRANSISTOR_PNPSMD
- added R1, R10, R11, R12, R13, R14, R15, R16, R17, R18, R19, R2, R20, R21, R22, R23, R24, R25, R26, R27, R28, R29, R3, R30, R31, R32, R33, R34, R4, R5, R6, R7, R8, R9: (no value), 1_SparkFun-Resistors:RESISTOR0603
- added U$1, U$10, U$100, U$101, U$102, U$103, U$104, U$105, U$106, U$107, U$108, U$109, U$11, U$110, U$111, U$112, U$113, U$114, U$115, U$116, U$117, U$118, U$119, U$12, U$120, U$121, U$122, U$123, U$124, U$125, U$126, U$127, U$128, U$129, U$13, U$130, U$131, U$132, U$133, U$134, U$135, U$136, U$137, U$138, U$139, U$14, U$140, U$141, U$142, U$143, U$144, U$145, U$146, U$147, U$148, U$149, U$15, U$150, U$151, U$152, U$153, U$154, U$155, U$156, U$157, U$158, U$159, U$16, U$160, U$161, U$162, U$163, U$164, U$165, U$166, U$167, U$168, U$169, U$17, U$170, U$171, U$172, U$173, U$174, U$175, U$176, U$177, U$178, U$179, U$18, U$180, U$181, U$182, U$183, U$184, U$185, U$186, U$187, U$188, U$189, U$19, U$190, U$191, U$192, U$193, U$194, U$195, U$196, U$197, U$198, U$199, U$2, U$20, U$200, U$201, U$202, U$203, U$204, U$205, U$206, U$207, U$208, U$209, U$21, U$210, U$211, U$212, U$213, U$214, U$215, U$216, U$217, U$218, U$219, U$22, U$220, U$221, U$222, U$223, U$224, U$225, U$226, U$227, U$228, U$229, U$23, U$230, U$231, U$232, U$233, U$234, U$235, U$236, U$237, U$238, U$239, U$24, U$240, U$241, U$242, U$243, U$244, U$245, U$246, U$247, U$248, U$249, U$25, U$250, U$251, U$252, U$253, U$254, U$255, U$256, U$257, U$26, U$27, U$28, U$29, U$3, U$30, U$31, U$32, U$33, U$34, U$35, U$36, U$37, U$38, U$39, U$4, U$40, U$41, U$42, U$43, U$44, U$45, U$46, U$47, U$48, U$49, U$50, U$51, U$52, U$53, U$54, U$55, U$56, U$57, U$58, U$59, U$6, U$60, U$61, U$62, U$63, U$64, U$65, U$66, U$67, U$68, U$69, U$7, U$70, U$71, U$72, U$73, U$74, U$75, U$76, U$77, U$78, U$79, U$8, U$80, U$81, U$82, U$83, U$84, U$85, U$86, U$87, U$88, U$89, U$9, U$90, U$91, U$92, U$93, U$94, U$95, U$96, U$97, U$98, U$99: PT15-21B, 0_Tristan's_Lib:PT15-21B
- added U$5: MUX-74HC4067SMD, 1_SparkFun-AnalogIC:MUX-74HC4067SMD
Connections:
- new net C1: IC2A.0, R19.1
- new net C10: IC2A.9, R28.1
- new net C11: IC2A.10, R29.1
- new net C12: IC2A.11, R30.1
- new net C13: IC2A.12, R31.1
- new net C14: IC2A.13, R32.1
- new net C15: IC2A.14, R33.1
- new net C16: IC2A.15, R34.1
- new net C2: IC2A.1, R20.1
- new net C3: IC2A.2, R21.1
- new net C4: IC2A.3, R22.1
- new net C5: IC2A.4, R23.1
- new net C6: IC2A.5, R24.1
- new net C7: IC2A.6, R25.1
- new net C8: IC2A.7, R26.1
- new net C9: IC2A.8, R27.1
- new net DIG_OUT: IC1G1.OUT1
- new net EN: U$5.EN
- new net GND: C1.-, C2.-, C3.-, C4.-, IC1G1.GND, IC2P.GND, R1.2, R10.2, R11.2, R12.2, R13.2, R14.2, R15.2, R16.2, R17.1, R2.2, R3.2, R4.2, R5.2, R6.2, R7.2, R8.2, R9.2, U$5.GND
- new net N$1: Q1.B, R19.2
- new net N$10: Q4.B, R22.2
- new net N$101: D49.C, U$50.C
- new net N$102: D50.C, U$51.C
- new net N$103: D52.C, U$53.C
- new net N$104: D51.C, U$52.C
- new net N$109: D53.C, U$54.C
- new net N$11: Q5.B, R23.2
- new net N$110: D54.C, U$55.C
- new net N$111: D56.C, U$57.C
- new net N$112: D55.C, U$56.C
- new net N$117: D57.C, U$58.C
- new net N$118: D58.C, U$59.C
- new net N$119: D60.C, U$61.C
- new net N$12: Q6.B, R24.2
- new net N$120: D59.C, U$60.C
- new net N$125: D61.C, U$62.C
- new net N$126: D62.C, U$63.C
- new net N$127: D64.C, U$65.C
- new net N$128: D63.C, U$64.C
- new net N$13: D5.C, U$6.C
- new net N$133: D65.C, U$66.C
- new net N$134: D66.C, U$67.C
- new net N$135: D68.C, U$69.C
- new net N$136: D67.C, U$68.C
- new net N$139: D69.C, U$70.C
- new net N$14: D6.C, U$7.C
- new net N$140: D70.C, U$71.C
- new net N$141: D72.C, U$73.C
- new net N$142: D71.C, U$72.C
- new net N$145: D73.C, U$74.C
- new net N$146: D74.C, U$75.C
- new net N$147: D76.C, U$77.C
- new net N$148: D75.C, U$76.C
- new net N$15: D8.C, U$9.C
- new net N$151: D77.C, U$78.C
- new net N$152: D78.C, U$79.C
- new net N$153: D80.C, U$81.C
- new net N$154: D79.C, U$80.C
- new net N$157: D81.C, U$82.C
- new net N$158: D82.C, U$83.C
- new net N$159: D84.C, U$85.C
- new net N$16: D7.C, U$8.C
- new net N$160: D83.C, U$84.C
- new net N$161: D85.C, U$86.C
- new net N$162: D86.C, U$87.C
- new net N$163: D88.C, U$89.C
- new net N$164: D87.C, U$88.C
- new net N$165: D89.C, U$90.C
- new net N$166: D90.C, U$91.C
- new net N$167: D92.C, U$93.C
- new net N$168: D91.C, U$92.C
- new net N$169: D93.C, U$94.C
- new net N$17: Q7.B, R25.2
- new net N$170: D94.C, U$95.C
- new net N$171: D96.C, U$97.C
- new net N$172: D95.C, U$96.C
- new net N$175: D97.C, U$98.C
- new net N$176: D98.C, U$99.C
- new net N$177: D100.C, U$101.C
- new net N$178: D99.C, U$100.C
- new net N$179: D101.C, U$102.C
- new net N$18: Q8.B, R26.2
- new net N$180: D102.C, U$103.C
- new net N$181: D104.C, U$105.C
- new net N$182: D103.C, U$104.C
- new net N$183: D105.C, U$106.C
- new net N$184: D106.C, U$107.C
- new net N$185: D108.C, U$109.C
- new net N$186: D107.C, U$108.C
- new net N$187: D109.C, U$110.C
- new net N$188: D110.C, U$111.C
- new net N$189: D112.C, U$113.C
- new net N$19: Q9.B, R27.2
- new net N$190: D111.C, U$112.C
- new net N$193: D113.C, U$114.C
- new net N$194: D114.C, U$115.C
- new net N$195: D116.C, U$117.C
- new net N$196: D115.C, U$116.C
- new net N$197: D117.C, U$118.C
- new net N$198: D118.C, U$119.C
- new net N$199: D120.C, U$121.C
- new net N$2: Q2.B, R20.2
- new net N$20: Q10.B, R28.2
- new net N$200: D119.C, U$120.C
- new net N$201: D121.C, U$122.C
- new net N$202: D122.C, U$123.C
- new net N$203: D124.C, U$125.C
- new net N$204: D123.C, U$124.C
- new net N$205: D125.C, U$126.C
- new net N$206: D126.C, U$127.C
- new net N$207: D128.C, U$129.C
- new net N$208: D127.C, U$128.C
- new net N$21: D9.C, U$10.C
- new net N$213: D129.C, U$130.C
- new net N$214: D130.C, U$131.C
- new net N$215: D132.C, U$133.C
- new net N$216: D131.C, U$132.C
- new net N$219: D133.C, U$134.C
- new net N$22: D10.C, U$11.C
- new net N$220: D134.C, U$135.C
- new net N$221: D136.C, U$137.C
- new net N$222: D135.C, U$136.C
- new net N$225: D137.C, U$138.C
- new net N$226: D138.C, U$139.C
- new net N$227: D140.C, U$141.C
- new net N$228: D139.C, U$140.C
- new net N$23: D12.C, U$13.C
- new net N$231: D141.C, U$142.C
- new net N$232: D142.C, U$143.C
- new net N$233: D144.C, U$145.C
- new net N$234: D143.C, U$144.C
- new net N$237: D145.C, U$146.C
- new net N$238: D146.C, U$147.C
- new net N$239: D148.C, U$149.C
- new net N$24: D11.C, U$12.C
- new net N$240: D147.C, U$148.C
- new net N$241: D149.C, U$150.C
- new net N$242: D150.C, U$151.C
- new net N$243: D152.C, U$153.C
- new net N$244: D151.C, U$152.C
- new net N$245: D153.C, U$154.C
- new net N$246: D154.C, U$155.C
- new net N$247: D156.C, U$157.C
- new net N$248: D155.C, U$156.C
- new net N$249: D157.C, U$158.C
- new net N$25: Q11.B, R29.2
- new net N$250: D158.C, U$159.C
- new net N$251: D160.C, U$161.C
- new net N$252: D159.C, U$160.C
- new net N$255: D161.C, U$162.C
- new net N$256: D162.C, U$163.C
- new net N$257: D164.C, U$165.C
- new net N$258: D163.C, U$164.C
- new net N$259: D165.C, U$166.C
- new net N$26: Q12.B, R30.2
- new net N$260: D166.C, U$167.C
- new net N$261: D168.C, U$169.C
- new net N$262: D167.C, U$168.C
- new net N$263: D169.C, U$170.C
- new net N$264: D170.C, U$171.C
- new net N$265: D172.C, U$173.C
- new net N$266: D171.C, U$172.C
- new net N$267: D173.C, U$174.C
- new net N$268: D174.C, U$175.C
- new net N$269: D176.C, U$177.C
- new net N$27: Q13.B, R31.2
- new net N$270: D175.C, U$176.C
- new net N$273: D177.C, U$178.C
- new net N$274: D178.C, U$179.C
- new net N$275: D180.C, U$181.C
- new net N$276: D179.C, U$180.C
- new net N$277: D181.C, U$182.C
- new net N$278: D182.C, U$183.C
- new net N$279: D184.C, U$185.C
- new net N$28: Q14.B, R32.2
- new net N$280: D183.C, U$184.C
- new net N$281: D185.C, U$186.C
- new net N$282: D186.C, U$187.C
- new net N$283: D188.C, U$189.C
- new net N$284: D187.C, U$188.C
- new net N$285: D189.C, U$190.C
- new net N$286: D190.C, U$191.C
- new net N$287: D192.C, U$193.C
- new net N$288: D191.C, U$192.C
- new net N$29: D13.C, U$14.C
- new net N$291: D193.C, U$194.C
- new net N$292: D194.C, U$195.C
- new net N$293: D196.C, U$197.C
- new net N$294: D195.C, U$196.C
- new net N$295: D197.C, U$198.C
- new net N$296: D198.C, U$199.C
- new net N$297: D200.C, U$201.C
- new net N$298: D199.C, U$200.C
- new net N$299: D201.C, U$202.C
- new net N$3: IC1G1.-IN1, U$5.COM
- new net N$30: D14.C, U$15.C
- new net N$300: D202.C, U$203.C
- new net N$301: D204.C, U$205.C
- new net N$302: D203.C, U$204.C
- new net N$303: D205.C, U$206.C
- new net N$304: D206.C, U$207.C
- new net N$305: D208.C, U$209.C
- new net N$306: D207.C, U$208.C
- new net N$309: D209.C, U$210.C
- new net N$31: D16.C, U$17.C
- new net N$310: D210.C, U$211.C
- new net N$311: D212.C, U$213.C
- new net N$312: D211.C, U$212.C
- new net N$313: D213.C, U$214.C
- new net N$314: D214.C, U$215.C
- new net N$315: D216.C, U$217.C
- new net N$316: D215.C, U$216.C
- new net N$317: D217.C, U$218.C
- new net N$318: D218.C, U$219.C
- new net N$319: D220.C, U$221.C
- new net N$32: D15.C, U$16.C
- new net N$320: D219.C, U$220.C
- new net N$321: D221.C, U$222.C
- new net N$322: D222.C, U$223.C
- new net N$323: D224.C, U$225.C
- new net N$324: D223.C, U$224.C
- new net N$327: D225.C, U$226.C
- new net N$328: D226.C, U$227.C
- new net N$329: D228.C, U$229.C
- new net N$33: Q15.B, R33.2
- new net N$330: D227.C, U$228.C
- new net N$331: D229.C, U$230.C
- new net N$332: D230.C, U$231.C
- new net N$333: D232.C, U$233.C
- new net N$334: D231.C, U$232.C
- new net N$335: D233.C, U$234.C
- new net N$336: D234.C, U$235.C
- new net N$337: D236.C, U$237.C
- new net N$338: D235.C, U$236.C
- new net N$339: D237.C, U$238.C
- new net N$34: Q16.B, R34.2
- new net N$340: D238.C, U$239.C
- new net N$341: D240.C, U$241.C
- new net N$342: D239.C, U$240.C
- new net N$345: D241.C, U$242.C
- new net N$346: D242.C, U$243.C
- new net N$347: D244.C, U$245.C
- new net N$348: D243.C, U$244.C
- new net N$349: D245.C, U$246.C
- new net N$350: D246.C, U$247.C
- new net N$351: D248.C, U$249.C
- new net N$352: D247.C, U$248.C
- new net N$353: D249.C, U$250.C
- new net N$354: D250.C, U$251.C
- new net N$355: D252.C, U$253.C
- new net N$356: D251.C, U$252.C
- new net N$357: D253.C, U$254.C
- new net N$358: D254.C, U$255.C
- new net N$359: D256.C, U$257.C
- new net N$360: D255.C, U$256.C
- new net N$37: D17.C, U$18.C
- new net N$38: D18.C, U$19.C
- new net N$39: D20.C, U$21.C
- new net N$4: D2.C, U$2.C
- new net N$40: D19.C, U$20.C
- new net N$45: D21.C, U$22.C
- new net N$46: D22.C, U$23.C
- new net N$47: D24.C, U$25.C
- new net N$48: D23.C, U$24.C
- new net N$5: C3.+, IC1G2.+IN2, R17.2, R18.1
- new net N$53: D25.C, U$26.C
- new net N$54: D26.C, U$27.C
- new net N$55: D28.C, U$29.C
- new net N$56: D27.C, U$28.C
- new net N$6: D1.C, U$1.C
- new net N$61: D29.C, U$30.C
- new net N$62: D30.C, U$31.C
- new net N$63: D32.C, U$33.C
- new net N$64: D31.C, U$32.C
- new net N$69: D33.C, U$34.C
- new net N$7: D4.C, U$4.C
- new net N$70: D34.C, U$35.C
- new net N$71: D36.C, U$37.C
- new net N$72: D35.C, U$36.C
- new net N$77: D37.C, U$38.C
- new net N$78: D38.C, U$39.C
- new net N$79: D40.C, U$41.C
- new net N$8: D3.C, U$3.C
- new net N$80: D39.C, U$40.C
- new net N$85: D41.C, U$42.C
- new net N$86: D42.C, U$43.C
- new net N$87: D44.C, U$45.C
- new net N$88: D43.C, U$44.C
- new net N$9: Q3.B, R21.2
- new net N$93: D45.C, U$46.C
- new net N$94: D46.C, U$47.C
- new net N$95: D48.C, U$49.C
- new net N$96: D47.C, U$48.C
- new net P1: D1.A, D100.A, D113.A, D116.A, D17.A, D20.A, D33.A, D36.A, D4.A, D49.A, D52.A, D65.A, D68.A, D81.A, D84.A, D97.A, Q1.C
- new net P10: D130.A, D131.A, D146.A, D147.A, D162.A, D163.A, D178.A, D179.A, D194.A, D195.A, D210.A, D211.A, D226.A, D227.A, D242.A, D243.A, Q10.C
- new net P11: D133.A, D136.A, D149.A, D152.A, D165.A, D168.A, D181.A, D184.A, D197.A, D200.A, D213.A, D216.A, D229.A, D232.A, D245.A, D248.A, Q11.C
- new net P12: D134.A, D135.A, D150.A, D151.A, D166.A, D167.A, D182.A, D183.A, D198.A, D199.A, D214.A, D215.A, D230.A, D231.A, D246.A, D247.A, Q12.C
- new net P13: D137.A, D140.A, D153.A, D156.A, D169.A, D172.A, D185.A, D188.A, D201.A, D204.A, D217.A, D220.A, D233.A, D236.A, D249.A, D252.A, Q13.C
- new net P14: D138.A, D139.A, D154.A, D155.A, D170.A, D171.A, D186.A, D187.A, D202.A, D203.A, D218.A, D219.A, D234.A, D235.A, D250.A, D251.A, Q14.C
- new net P15: D141.A, D144.A, D157.A, D160.A, D173.A, D176.A, D189.A, D192.A, D205.A, D208.A, D221.A, D224.A, D237.A, D240.A, D253.A, D256.A, Q15.C
- new net P16: D142.A, D143.A, D158.A, D159.A, D174.A, D175.A, D190.A, D191.A, D206.A, D207.A, D222.A, D223.A, D238.A, D239.A, D254.A, D255.A, Q16.C
- new net P2: D114.A, D115.A, D18.A, D19.A, D2.A, D3.A, D34.A, D35.A, D50.A, D51.A, D66.A, D67.A, D82.A, D83.A, D98.A, D99.A, Q2.C
- new net P3: D101.A, D104.A, D117.A, D120.A, D21.A, D24.A, D37.A, D40.A, D5.A, D53.A, D56.A, D69.A, D72.A, D8.A, D85.A, D88.A, Q3.C
- new net P4: D102.A, D103.A, D118.A, D119.A, D22.A, D23.A, D38.A, D39.A, D54.A, D55.A, D6.A, D7.A, D70.A, D71.A, D86.A, D87.A, Q4.C
- new net P5: D105.A, D108.A, D12.A, D121.A, D124.A, D25.A, D28.A, D41.A, D44.A, D57.A, D60.A, D73.A, D76.A, D89.A, D9.A, D92.A, Q5.C
- new net P6: D10.A, D106.A, D107.A, D11.A, D122.A, D123.A, D26.A, D27.A, D42.A, D43.A, D58.A, D59.A, D74.A, D75.A, D90.A, D91.A, Q6.C
- new net P7: D109.A, D112.A, D125.A, D128.A, D13.A, D16.A, D29.A, D32.A, D45.A, D48.A, D61.A, D64.A, D77.A, D80.A, D93.A, D96.A, Q7.C
- new net P8: D110.A, D111.A, D126.A, D127.A, D14.A, D15.A, D30.A, D31.A, D46.A, D47.A, D62.A, D63.A, D78.A, D79.A, D94.A, D95.A, Q8.C
- new net P9: D129.A, D132.A, D145.A, D148.A, D161.A, D164.A, D177.A, D180.A, D193.A, D196.A, D209.A, D212.A, D225.A, D228.A, D241.A, D244.A, Q9.C
- new net S1: U$5.S0
- new net S2: U$5.S1
- new net S3: U$5.S2
- new net S4: U$5.S3
- new net S5: IC2A.A
- new net S6: IC2A.B
- new net S7: IC2A.C
- new net S8: IC2A.D
- new net THRESHOLD: IC1G1.+IN1, IC1G2.-IN2, IC1G2.OUT2
- new net VCC: C1.+, C2.+, C4.+, IC1G1.+V, IC2P.VCC, Q1.E, Q10.E, Q11.E, Q12.E, Q13.E, Q14.E, Q15.E, Q16.E, Q2.E, Q3.E, Q4.E, Q5.E, Q6.E, Q7.E, Q8.E, Q9.E, R18.2, U$5.VCC
- new net Y1: R1.1, U$114.E, U$115.E, U$118.E, U$119.E, U$122.E, U$123.E, U$126.E, U$127.E, U$242.E, U$243.E, U$246.E, U$247.E, U$250.E, U$251.E, U$254.E, U$255.E, U$5.CHAN0
- new net Y10: R10.1, U$180.E, U$181.E, U$184.E, U$185.E, U$188.E, U$189.E, U$192.E, U$193.E, U$5.CHAN9, U$52.E, U$53.E, U$56.E, U$57.E, U$60.E, U$61.E, U$64.E, U$65.E
- new net Y11: R11.1, U$162.E, U$163.E, U$166.E, U$167.E, U$170.E, U$171.E, U$174.E, U$175.E, U$34.E, U$35.E, U$38.E, U$39.E, U$42.E, U$43.E, U$46.E, U$47.E, U$5.CHAN10
- new net Y12: R12.1, U$164.E, U$165.E, U$168.E, U$169.E, U$172.E, U$173.E, U$176.E, U$177.E, U$36.E, U$37.E, U$40.E, U$41.E, U$44.E, U$45.E, U$48.E, U$49.E, U$5.CHAN11
- new net Y13: R13.1, U$146.E, U$147.E, U$150.E, U$151.E, U$154.E, U$155.E, U$158.E, U$159.E, U$18.E, U$19.E, U$22.E, U$23.E, U$26.E, U$27.E, U$30.E, U$31.E, U$5.CHAN12
- new net Y14: R14.1, U$148.E, U$149.E, U$152.E, U$153.E, U$156.E, U$157.E, U$160.E, U$161.E, U$20.E, U$21.E, U$24.E, U$25.E, U$28.E, U$29.E, U$32.E, U$33.E, U$5.CHAN13
- new net Y15: R15.1, U$1.E, U$10.E, U$11.E, U$130.E, U$131.E, U$134.E, U$135.E, U$138.E, U$139.E, U$14.E, U$142.E, U$143.E, U$15.E, U$2.E, U$5.CHAN14, U$6.E, U$7.E
- new net Y16: R16.1, U$12.E, U$13.E, U$132.E, U$133.E, U$136.E, U$137.E, U$140.E, U$141.E, U$144.E, U$145.E, U$16.E, U$17.E, U$3.E, U$4.E, U$5.CHAN15, U$8.E, U$9.E
- new net Y2: R2.1, U$116.E, U$117.E, U$120.E, U$121.E, U$124.E, U$125.E, U$128.E, U$129.E, U$244.E, U$245.E, U$248.E, U$249.E, U$252.E, U$253.E, U$256.E, U$257.E, U$5.CHAN1
- new net Y3: R3.1, U$102.E, U$103.E, U$106.E, U$107.E, U$110.E, U$111.E, U$226.E, U$227.E, U$230.E, U$231.E, U$234.E, U$235.E, U$238.E, U$239.E, U$5.CHAN2, U$98.E, U$99.E
- new net Y4: R4.1, U$100.E, U$101.E, U$104.E, U$105.E, U$108.E, U$109.E, U$112.E, U$113.E, U$228.E, U$229.E, U$232.E, U$233.E, U$236.E, U$237.E, U$240.E, U$241.E, U$5.CHAN3
- new net Y5: R5.1, U$210.E, U$211.E, U$214.E, U$215.E, U$218.E, U$219.E, U$222.E, U$223.E, U$5.CHAN4, U$82.E, U$83.E, U$86.E, U$87.E, U$90.E, U$91.E, U$94.E, U$95.E
- new net Y6: R6.1, U$212.E, U$213.E, U$216.E, U$217.E, U$220.E, U$221.E, U$224.E, U$225.E, U$5.CHAN5, U$84.E, U$85.E, U$88.E, U$89.E, U$92.E, U$93.E, U$96.E, U$97.E
- new net Y7: R7.1, U$194.E, U$195.E, U$198.E, U$199.E, U$202.E, U$203.E, U$206.E, U$207.E, U$5.CHAN6, U$66.E, U$67.E, U$70.E, U$71.E, U$74.E, U$75.E, U$78.E, U$79.E
- new net Y8: R8.1, U$196.E, U$197.E, U$200.E, U$201.E, U$204.E, U$205.E, U$208.E, U$209.E, U$5.CHAN7, U$68.E, U$69.E, U$72.E, U$73.E, U$76.E, U$77.E, U$80.E, U$81.E
- new net Y9: R9.1, U$178.E, U$179.E, U$182.E, U$183.E, U$186.E, U$187.E, U$190.E, U$191.E, U$5.CHAN8, U$50.E, U$51.E, U$54.E, U$55.E, U$58.E, U$59.E, U$62.E, U$63.E
